File: Flaps&Spedd.kicad_pcb (KiCad board)
At the start: 2 copper layers, 46 x 46 mm, 22 parts, among them J1 CAN-M, J2 CAN-F, U1 SN65HVD230

Commit message: v3
Parts:
- removed H1: 5V, Connector_PinHeader_1.00mm:PinHeader_1x01_P1.00mm_Vertical
- removed H10, H11, H12, H13, H14, H7, H8, H9: 1, Connector_PinHeader_1.00mm:PinHeader_1x01_P1.00mm_Vertical
- removed H2, H3: GND, Connector_PinHeader_1.00mm:PinHeader_1x01_P1.00mm_Vertical
- removed H4: 12V, Connector_PinHeader_1.00mm:PinHeader_1x01_P1.00mm_Vertical
- added C2: 100pF, Resistor_SMD:R_1206_3216Metric_Pad1.30x1.75mm_HandSolder, F.Cu at (71.5, 89.0)
- added C3: 100pF, Resistor_SMD:R_1206_3216Metric_Pad1.30x1.75mm_HandSolder, F.Cu at (71.5, 79.0)
- added J3: Conn_01x08_Pin, Connector_PinSocket_2.54mm:PinSocket_1x08_P2.54mm_Vertical, F.Cu at (57.1, 67.3)
- added J4: Conn_01x04_Pin, Connector_PinSocket_2.54mm:PinSocket_1x04_P2.54mm_Vertical, F.Cu at (65.7, 73.4)
- added L1: ACT1210-220-2P-TL00, Filter:ACT1210_TDK, F.Cu at (73.0, 84.0)
- C1: footprint Connector_PinHeader_1.00mm:PinHeader_1x01_P1.00mm_Vertical -> Resistor_SMD:R_1206_3216Metric_Pad1.30x1.75mm_HandSolder
- J1: value CAN-M -> CAN-In
- J2: value CAN-F -> CAN-Out
- R1, R2: footprint Resistor_SMD:R_0805_2012Metric -> Resistor_SMD:R_1206_3216Metric_Pad1.30x1.75mm_HandSolder
- moved JP1 19.9 mm to (89.5, 81.2), turned to 90 degrees
- moved R2 17.6 mm to (89.5, 76.0), turned to 90 degrees
- moved C1 3.85 mm to (62.5, 79.0), turned to 180 degrees
- moved U1 3.08 mm to (64.3, 83.9)
- moved R1 2.14 mm to (67.5, 78.0), turned to 90 degrees
- moved MH3 0.52 mm to (94.5, 76.2)
Connections:
- U1 pad 6: Net-(J1-Pin_5) -> Net-(U1-CANL)
- U1 pad 7: Net-(J1-Pin_4) -> Net-(U1-CANH)
Routing:
- net GND: track 63.3 -> 0.00 mm, vias 0 -> 13
- net Net-(J1-Pin_1): track 22.9 -> 38.2 mm, vias 0 -> 1
- net Net-(J1-Pin_5): track 53.7 -> 38.7 mm
- net Net-(J3-Pin_1): track 0.00 -> 13.3 mm
- net Net-(H1-Pad1): track 13.0 -> 0.00 mm
- net Net-(U1-CANH): track 0.00 -> 7.78 mm
- net Net-(U1-CANL): track 0.00 -> 7.68 mm
- net Net-(JP1-B): track 7.67 -> 2.90 mm
- net Net-(J3-Pin_7): track 8.35 -> 4.96 mm
- net Net-(J3-Pin_8): track 8.28 -> 5.01 mm
- net +12V: track 32.8 -> 36.0 mm
- net Net-(J1-Pin_4): track 37.6 -> 34.7 mm
- net +3V3: track 16.7 -> 19.2 mm
- net Net-(U1-Rs): track 4.09 -> 2.75 mm
- added copper zone on B.Cu, net GND
- added copper zone on F.Cu, net GND
Other:
- board text added: "v3"
- board text removed: "v2"
